File: schematics/schematic/schematic.sch (KiCad schematic (older format))
At the start: 7 parts

Commit message: full schematic
Parts:
- added Brd?: SSD1306, symbol SSD1306-128x64_OLED:SSD1306
- added SW?: Rotary_Encoder_Switch, symbol Device:Rotary_Encoder_Switch
Connections:
- wire segments 48 -> 73
Changed lines of the file:
@@
 	4450 3000 5050 3000
 Wire Wire Line
-	5050 3000 5050 1300
+	9050 2450 9850 2450
+$Comp
+L Device:Rotary_Encoder_Switch SW?
+U 1 1 613C7F9F
+P 4750 1000
+F 0 "SW?" H 4750 1367 50  0000 C CNN
+F 1 "Rotary_Encoder_Switch" H 4750 1276 50  0000 C CNN
+F 2 "" H 4600 1160 50  0001 C CNN
+F 3 "~" H 4750 1260 50  0001 C CNN
+	1    4750 1000
+	1    0    0    -1
+$EndComp
 Wire Wire Line
-	5050 1300 9850 1300
+	5050 1900 5900 1900
 Wire Wire Line
-	9050 2450 9850 2450
+	5900 1900 5900 1350
 Wire Wire Line
-	9850 1300 9850 2450
+	5900 1350 9850 1350
+Wire Wire Line
+	9850 1350 9850 2450
+$Comp
+L power:GND #PWR?
+U 1 1 613D740B
+P 5150 1150
+F 0 "#PWR?" H 5150 900 50  0001 C CNN
+F 1 "GND" H 5155 977 50  0000 C CNN
+F 2 "" H 5150 1150 50  0001 C CNN
+F 3 "" H 5150 1150 50  0001 C CNN
+	1    5150 1150
+	1    0    0    -1
+$EndComp
+$Comp
+L power:GND #PWR?
+U 1 1 613D7CF3
+P 4250 1000
+F 0 "#PWR?" H 4250 750 50  0001 C CNN
+F 1 "GND" H 4255 827 50  0000 C CNN
+F 2 "" H 4250 1000 50  0001 C CNN
+F 3 "" H 4250 1000 50  0001 C CNN
+	1    4250 1000
+	1    0    0    -1
+$EndComp
+Wire Wire Line
+	4250 1000 4450 1000
+Wire Wire Line
+	5150 1150 5150 1100
+Wire Wire Line
+	5150 1100 5050 1100
+Wire Wire Line
+	5100 900  5250 900
+Wire Wire Line
+	5250 900  5250 2100
+Wire Wire Line
+	5250 2100 5200 2100
+Wire Wire Line
+	5200 2100 5200 3100
+Wire Wire Line
+	5200 3100 4450 3100
+Wire Wire Line
+	5050 1900 5050 3000
+Wire Wire Line
+	4450 1100 4450 1300
+Wire Wire Line
+	4450 1300 4750 1300
+Wire Wire Line
+	4750 1300 4750 3300
+Wire Wire Line
+	4750 3300 4450 3300
+Wire Wire Line
+	4450 900  4400 900
+Wire Wire Line
+	4400 900  4400 1650
+Wire Wire Line
+	4400 1650 4600 1650
+Wire Wire Line
+	4600 1650 4600 3200
+Wire Wire Line
+	4600 3200 4450 3200
+$Comp
+L SSD1306-128x64_OLED:SSD1306 Brd?
+U 1 1 613E7218
+P 1900 3550
+F 0 "Brd?" V 1485 3608 50  0000 C CNN
+F 1 "SSD1306" V 1576 3608 50  0000 C CNN
+F 2 "" H 1900 3800 50  0001 C CNN
+F 3 "" H 1900 3800 50  0001 C CNN
+	1    1900 3550
+	0    1    1    0
+$EndComp
+Wire Wire Line
+	2250 3700 3150 3700
+Wire Wire Line
+	2250 3600 3150 3600
+$Comp
+L power:GND #PWR?
+U 1 1 613FACF4
+P 2200 3000
+F 0 "#PWR?" H 2200 2750 50  0001 C CNN
+F 1 "GND" H 2250 3100 50  0000 C CNN
+F 2 "" H 2200 3000 50  0001 C CNN
+F 3 "" H 2200 3000 50  0001 C CNN
+	1    2200 3000
+	1    0    0    -1
+$EndComp
+Wire Wire Line
+	2250 3500 2550 3500
+Wire Wire Line
+	2550 3500 2550 3000
+Wire Wire Line
+	2250 3400 2250 3000
+Wire Wire Line
+	2250 3000 2200 3000
+$Comp
+L power:+3.3V #PWR?
+U 1 1 613FBE61
+P 2550 3000
+F 0 "#PWR?" H 2550 2850 50  0001 C CNN
+F 1 "+3.3V" H 2565 3173 50  0000 C CNN
+F 2 "" H 2550 3000 50  0001 C CNN
+F 3 "" H 2550 3000 50  0001 C CNN
+	1    2550 3000
+	1    0    0    -1
+$EndComp
 $EndSCHEMATC
